Commit message: added rplidar

File: scout_description/urdf/scout_v2/scout_v2.xacro (robot description, xacro)
@@ -55,4 +55,17 @@
         <child link="inertial_link" />
     </joint>
+  <link name="rplidar_link">
+    <visual>
+      <origin xyz="0 0 0" rpy="0 0 0">
+      <geometry>
+        <cylinder length="0.06" radius="0.005"/>
+      </geometry>
+    </visual>
+  </link>
+  <joint name="rplidar_joint" type="fixed">
+    <parent link="base_link"/>
+    <child link="rplidar_link"/>
+    <origin xyz="0.15 0.0 0.20" rpy="0 0 0"/>
+  </joint>
     <!-- Scout wheel macros -->
     <!-- wheel labeled from 0 to 3, conter-clockwise, starting from front right wheel -->

Commit message: added in more lidar stuff into gazebo as well as the scout v2 xacro

File: scout_description/urdf/scout_v2/scout_v2.xacro (robot description, xacro)
@@ -55,17 +55,17 @@
         <child link="inertial_link" />
     </joint>
-  <link name="rplidar_link">
-    <visual>
-      <origin xyz="0 0 0" rpy="0 0 0">
-      <geometry>
-        <cylinder length="0.06" radius="0.005"/>
-      </geometry>
-    </visual>
-  </link>
-  <joint name="rplidar_joint" type="fixed">
-    <parent link="base_link"/>
-    <child link="rplidar_link"/>
-    <origin xyz="0.15 0.0 0.20" rpy="0 0 0"/>
-  </joint>
+    <link name="rplidar_link">
+        <visual>
+            <origin xyz="0 0 0" rpy="0 0 0" />
+            <geometry>
+                <cylinder length="0.06" radius="0.005" />
+            </geometry>
+        </visual>
+    </link>
+    <joint name="rplidar_joint" type="fixed">
+        <parent link="base_link" />
+        <child link="rplidar_link" />
+        <origin xyz="0.3 0.0 0.20" rpy="0 0 0" />
+    </joint>
     <!-- Scout wheel macros -->
     <!-- wheel labeled from 0 to 3, conter-clockwise, starting from front right wheel -->

File: scout_description/urdf/scout_v2/scout_v2_gazebo.xacro (robot description, xacro)
@@ -28,3 +28,33 @@
     </plugin>
   </gazebo>
+  <gazebo reference="rplidar_link">
+    <sensor name="rplidar" type="gpu_lidar">
+      <pose>0 0 0 0 0 0</pose>
+      <topic>/scan</topic>
+      <update_rate>40</update_rate>
+      <ray>
+        <scan>
+          <horizontal>
+            <samples>720</samples>
+            <resolution>1</resolution>
+            <min_angle>-3.14159</min_angle>
+            <max_angle>3.14159</max_angle>
+          </horizontal>
+        </scan>
+        <range>
+          <min>0.2</min>
+          <max>15.0</max>
+          <resolution>0.01</resolution>
+        </range>
+        <noise>
+          <type>gaussian</type>
+          <mean>0.0</mean>
+          <stddev>0.01</stddev>
+        </noise>
+      </ray>
+      <always_on>true</always_on>
+      <visualize>true</visualize>
+      <gz_frame_id>rplidar_link</gz_frame_id>
+    </sensor>
+  </gazebo>
 </robot>

Commit message: updated tf postion

File: scout_description/urdf/scout_v2/scout_v2.xacro (robot description, xacro)
@@ -56,15 +56,38 @@
     </joint>
     <link name="rplidar_link">
+        <inertial>
+            <mass value="0.19" />
+            <origin xyz="0 0 0" />
+            <inertia ixx="0.00012" ixy="0" ixz="0" iyy="0.00012" iyz="0" izz="0.00018" />
+        </inertial>
         <visual>
-            <origin xyz="0 0 0" rpy="0 0 0" />
+            <origin xyz="0 0 0.02" rpy="0 0 0" />
             <geometry>
-                <cylinder length="0.06" radius="0.005" />
+                <cylinder length="0.04" radius="0.04" />
             </geometry>
+            <material name="rplidar_black">
+                <color rgba="0.02 0.02 0.02 1.0" />
+            </material>
         </visual>
+        <visual>
+            <origin xyz="0 0 0.045" rpy="0 0 0" />
+            <geometry>
+                <cylinder length="0.01" radius="0.032" />
+            </geometry>
+            <material name="rplidar_cap">
+                <color rgba="0.10 0.10 0.10 1.0" />
+            </material>
+        </visual>
+        <collision>
+            <origin xyz="0 0 0.02" rpy="0 0 0" />
+            <geometry>
+                <cylinder length="0.04" radius="0.04" />
+            </geometry>
+        </collision>
     </link>
     <joint name="rplidar_joint" type="fixed">
         <parent link="base_link" />
         <child link="rplidar_link" />
-        <origin xyz="0.3 0.0 0.20" rpy="0 0 0" />
+        <origin xyz="-0.28 0.0 0.3" rpy="0 0 0" />
     </joint>
     <!-- Scout wheel macros -->

File: scout_description/urdf/scout_v2/scout_v2_gazebo.xacro (robot description, xacro)
@@ -29,4 +29,5 @@
   </gazebo>
   <gazebo reference="rplidar_link">
+    <material>Gazebo/Black</material>
     <sensor name="rplidar" type="gpu_lidar">
       <pose>0 0 0 0 0 0</pose>

Commit message: 1. RViz fixed frame map → odom (no map server in this launch) 2. Lidar frame - URDF now uses laser frame at (0.20, 0, 0.20) matching your hardware, removed redundant static TF publisher 3. Wheel TFs - Added joint_state_publisher to publish joint states for the continuous wheel joints

File: scout_description/urdf/scout_v2/scout_v2.xacro (robot description, xacro)
@@ -55,5 +55,5 @@
         <child link="inertial_link" />
     </joint>
-    <link name="rplidar_link">
+    <link name="laser">
         <inertial>
             <mass value="0.19" />
@@ -88,6 +88,6 @@
     <joint name="rplidar_joint" type="fixed">
         <parent link="base_link" />
-        <child link="rplidar_link" />
-        <origin xyz="-0.28 0.0 0.3" rpy="0 0 0" />
+        <child link="laser" />
+        <origin xyz="0.20 0.0 0.20" rpy="0 0 0" />
     </joint>
     <!-- Scout wheel macros -->

Commit message: got robot to move once every 20s

File: scout_description/urdf/scout_v2/scout_v2.xacro (robot description, xacro)
@@ -89,5 +89,5 @@
         <parent link="base_link" />
         <child link="laser" />
-        <origin xyz="0.20 0.0 0.20" rpy="0 0 0" />
+        <origin xyz="-0.23 0.0 0.45" rpy="0 0 0" />
     </joint>
     <!-- Scout wheel macros -->

Commit message: added lidar rotation

File: scout_description/urdf/scout_v2/scout_v2.xacro (robot description, xacro)
@@ -89,5 +89,5 @@
         <parent link="base_link" />
         <child link="laser" />
-        <origin xyz="-0.23 0.0 0.45" rpy="0 0 0" />
+        <origin xyz="-0.23 0.0 0.45" rpy="0 0 3.1416"/>
     </joint>
     <!-- Scout wheel macros -->
